File: KiCAD/FV-1_Test_Board/FV-1_Test_Board.kicad_pcb (KiCad board)
At the start: 2 copper layers, 94 x 71.1 mm, 32 parts, among them J1 PWR, J2 LOUT, J3 ROUT, J4 IN, J5 TP_GND, J6 S0, J7 S1, J8 S2, U1 AE-FV-1-DIP_large

Commit message: Interface Board
Parts:
- removed R7: 1k C&T, Resistor_THT:R_Axial_DIN0207_L6.3mm_D2.5mm_P10.16mm_Horizontal
- added D2: 1S4, Diode_THT:D_DO-35_SOD27_P10.16mm_Horizontal, F.Cu at (142.2, 83.8)
- added D3: 1S4, Diode_THT:D_DO-35_SOD27_P10.16mm_Horizontal, F.Cu at (129.5, 88.9)
- added G***: LOGO, myfootprint:Silk_PNPN_Manufactory_400dpi, F.Cu at (116.3, 125.7)
- C7: value 0.047u -> 1000p
Routing:
- net +3V3: track 68.6 -> 91.4 mm
- net Net-(C7-Pad1): track 17.8 -> 20.3 mm
