File: KiCAD/FV-1_Test_Board/FV-1_Test_Board.sch (KiCad schematic (older format))
At the start: 32 parts, among them J1 PWR, J2 LOUT, J3 ROUT, J4 IN, J5 TP_GND, J6 S0, J7 S1, J8 S2, U1 AE-FV-1-DIP_large

Commit message: Interface Board
Parts:
- removed R7: 1k C&T, Resistor_THT:R_Axial_DIN0207_L6.3mm_D2.5mm_P10.16mm_Horizontal, symbol Device:R
- added D2, D3: 1S4, Diode_THT:D_DO-35_SOD27_P10.16mm_Horizontal, symbol Device:D_Schottky
- C7: value 0.047u -> 0.047uF
Connections:
- wire segments 99 -> 101
Other:
- moved on the sheet: C6, C7, J4, R6
Changed lines of the file:
@@
 Sheet 1 1
 Title "FV-1 Test Board"
-Date "2021-08-04"
+Date "2021-08-22"
 Rev "Ver. 1.0"
 Comp "PNPN Manufactory"
@@
 L Connector_Generic:Conn_01x02 J4
 U 1 1 60D3E6F3
-P 3500 3150
-F 0 "J4" H 3418 3367 50  0000 C CNN
-F 1 "IN" H 3418 3276 50  0000 C CNN
-F 2 "Connector_PinHeader_2.54mm:PinHeader_1x02_P2.54mm_Vertical" H 3500 3150 50  0001 C CNN
-F 3 "~" H 3500 3150 50  0001 C CNN
-	1    3500 3150
+P 3300 3150
+F 0 "J4" H 3218 3367 50  0000 C CNN
+F 1 "IN" H 3218 3276 50  0000 C CNN
+F 2 "Connector_PinHeader_2.54mm:PinHeader_1x02_P2.54mm_Vertical" H 3300 3150 50  0001 C CNN
+F 3 "~" H 3300 3150 50  0001 C CNN
+	1    3300 3150
 	-1   0    0    -1
 $EndComp
@@
 L Device:C C6
 U 1 1 60D3EB99
-P 3900 3150
-F 0 "C6" V 3648 3150 50  0000 C CNN
-F 1 "1u" V 3739 3150 50  0000 C CNN
-F 2 "Capacitor_THT:C_Rect_L7.0mm_W4.5mm_P5.00mm" H 3938 3000 50  0001 C CNN
-F 3 "~" H 3900 3150 50  0001 C CNN
-	1    3900 3150
+P 3700 3150
+F 0 "C6" V 3448 3150 50  0000 C CNN
+F 1 "1u" V 3539 3150 50  0000 C CNN
+F 2 "Capacitor_THT:C_Rect_L7.0mm_W4.5mm_P5.00mm" H 3738 3000 50  0001 C CNN
+F 3 "~" H 3700 3150 50  0001 C CNN
+	1    3700 3150
 	0    1    1    0
 $EndComp
@@
 L Device:R R6
 U 1 1 60D3F810
-P 4250 3150
-F 0 "R6" V 4043 3150 50  0000 C CNN
-F 1 "1k" V 4134 3150 50  0000 C CNN
-F 2 "Resistor_THT:R_Axial_DIN0207_L6.3mm_D2.5mm_P10.16mm_Horizontal" V 4180 3150 50  0001 C CNN
-F 3 "~" H 4250 3150 50  0001 C CNN
-	1    4250 3150
+P 4050 3150
+F 0 "R6" V 3843 3150 50  0000 C CNN
+F 1 "1k" V 3934 3150 50  0000 C CNN
+F 2 "Resistor_THT:R_Axial_DIN0207_L6.3mm_D2.5mm_P10.16mm_Horizontal" V 3980 3150 50  0001 C CNN
+F 3 "~" H 4050 3150 50  0001 C CNN
+	1    4050 3150
 	0    1    1    0
 $EndComp
@@
 L Device:C C7
 U 1 1 60D3FD2B
-P 4850 3400
-F 0 "C7" H 4965 3446 50  0000 L CNN
-F 1 "0.047u" H 4965 3355 50  0000 L CNN
-F 2 "Capacitor_THT:C_Rect_L7.0mm_W3.5mm_P5.00mm" H 4888 3250 50  0001 C CNN
-F 3 "~" H 4850 3400 50  0001 C CNN
-	1    4850 3400
+P 4750 3400
+F 0 "C7" H 4865 3446 50  0000 L CNN
+F 1 "0.047uF" H 4865 3355 50  0000 L CNN
+F 2 "Capacitor_THT:C_Rect_L7.0mm_W3.5mm_P5.00mm" H 4788 3250 50  0001 C CNN
+F 3 "~" H 4750 3400 50  0001 C CNN
+	1    4750 3400
 	1    0    0    -1
 $EndComp
@@
 $EndComp
 Wire Wire Line
-	3700 3150 3750 3150
-Wire Wire Line
-	4050 3150 4100 3150
-Wire Wire Line
-	4400 3150 4500 3150
-Wire Wire Line
-	4850 3150 4850 3250
-Connection ~ 4850 3150
+	3500 3150 3550 3150
+Wire Wire Line
+	3850 3150 3900 3150
+Wire Wire Line
+	4200 3150 4400 3150
+Wire Wire Line
+	4750 3150 4750 3250
+Connection ~ 4750 3150
 Wire Wire Line
 	5500 3150 5450 3150
@@
 L power:GND #PWR014
 U 1 1 60D44F9F
-P 4850 3600
-F 0 "#PWR014" H 4850 3350 50  0001 C CNN
-F 1 "GND" H 4855 3427 50  0000 C CNN
-F 2 "" H 4850 3600 50  0001 C CNN
-F 3 "" H 4850 3600 50  0001 C CNN
-	1    4850 3600
+P 4750 3600
+F 0 "#PWR014" H 4750 3350 50  0001 C CNN
+F 1 "GND" H 4755 3427 50  0000 C CNN
+F 2 "" H 4750 3600 50  0001 C CNN
+F 3 "" H 4750 3600 50  0001 C CNN
+	1    4750 3600
 	1    0    0    -1
 $EndComp
@@
 L power:GND #PWR012
 U 1 1 60D4552A
-P 3750 3600
-F 0 "#PWR012" H 3750 3350 50  0001 C CNN
-F 1 "GND" H 3755 3427 50  0000 C CNN
-F 2 "" H 3750 3600 50  0001 C CNN
-F 3 "" H 3750 3600 50  0001 C CNN
-	1    3750 3600
-	1    0    0    -1
-$EndComp
-Wire Wire Line
-	3700 3250 3750 3250
-Wire Wire Line
-	3750 3250 3750 3600
-Wire Wire Line
-	4850 3600 4850 3550
+P 3550 3600
+F 0 "#PWR012" H 3550 3350 50  0001 C CNN
+F 1 "GND" H 3555 3427 50  0000 C CNN
+F 2 "" H 3550 3600 50  0001 C CNN
+F 3 "" H 3550 3600 50  0001 C CNN
+	1    3550 3600
+	1    0    0    -1
+$EndComp
+Wire Wire Line
+	3500 3250 3550 3250
+Wire Wire Line
+	3550 3250 3550 3600
+Wire Wire Line
+	4750 3600 4750 3550
 $Comp
 L power:+3V3 #PWR016
@@
 Connection ~ 5450 3150
 Wire Wire Line
-	5450 3150 4850 3150
+	5450 3150 4750 3150
 Wire Wire Line
 	5450 3650 5500 3650
@@
 L power:GND #PWR013
 U 1 1 60E5FCE3
-P 4500 3600
-F 0 "#PWR013" H 4500 3350 50  0001 C CNN
-F 1 "GND" H 4505 3427 50  0000 C CNN
-F 2 "" H 4500 3600 50  0001 C CNN
-F 3 "" H 4500 3600 50  0001 C CNN
-	1    4500 3600
-	1    0    0    -1
-$EndComp
-Wire Wire Line
-	4500 3250 4500 3150
-Connection ~ 4500 3150
-Wire Wire Line
-	4500 3150 4850 3150
-Wire Wire Line
-	4500 3600 4500 3550
+P 4400 3600
+F 0 "#PWR013" H 4400 3350 50  0001 C CNN
+F 1 "GND" H 4405 3427 50  0000 C CNN
+F 2 "" H 4400 3600 50  0001 C CNN
+F 3 "" H 4400 3600 50  0001 C CNN
+	1    4400 3600
+	1    0    0    -1
+$EndComp
+Wire Wire Line
+	4400 3250 4400 3150
+Connection ~ 4400 3150
+Wire Wire Line
+	4400 3150 4750 3150
+Wire Wire Line
+	4400 3600 4400 3550
 NoConn ~ 5500 4900
 NoConn ~ 5500 5150
-$Comp
-L Device:R R7
-U 1 1 60E5F39B
-P 4500 3400
-F 0 "R7" H 4300 3450 50  0000 L CNN
-F 1 "1k C&T" H 4150 3350 50  0000 L CNN
-F 2 "Resistor_THT:R_Axial_DIN0207_L6.3mm_D2.5mm_P10.16mm_Horizontal" V 4430 3400 50  0001 C CNN
-F 3 "~" H 4500 3400 50  0001 C CNN
-	1    4500 3400
-	1    0    0    -1
-$EndComp
 $Comp
 L Connector_Generic:Conn_01x02 J1
@@
 	1    0    0    -1
 $EndComp
+$Comp
+L Device:D_Schottky D3
+U 1 1 611C007F
+P 4400 3400
+F 0 "D3" V 4350 3200 50  0000 L CNN
+F 1 "1S4" V 4450 3150 50  0000 L CNN
+F 2 "Diode_THT:D_DO-35_SOD27_P10.16mm_Horizontal" H 4400 3400 50  0001 C CNN
+F 3 "~" H 4400 3400 50  0001 C CNN
+	1    4400 3400
+	0    1    1    0
+$EndComp
+Wire Wire Line
+	4400 3000 4400 3150
+Wire Wire Line
+	4400 2700 4400 2650
+$Comp
+L power:+3V3 #PWR024
+U 1 1 611E1B8D
+P 4400 2650
+F 0 "#PWR024" H 4400 2500 50  0001 C CNN
+F 1 "+3V3" H 4415 2823 50  0000 C CNN
+F 2 "" H 4400 2650 50  0001 C CNN
+F 3 "" H 4400 2650 50  0001 C CNN
+	1    4400 2650
+	1    0    0    -1
+$EndComp
+$Comp
+L Device:D_Schottky D2
+U 1 1 611D7F98
+P 4400 2850
+F 0 "D2" V 4350 2650 50  0000 L CNN
+F 1 "1S4" V 4450 2600 50  0000 L CNN
+F 2 "Diode_THT:D_DO-35_SOD27_P10.16mm_Horizontal" H 4400 2850 50  0001 C CNN
+F 3 "~" H 4400 2850 50  0001 C CNN
+	1    4400 2850
+	0    1    1    0
+$EndComp
 $EndSCHEMATC
