File: KiCAD/FV-1_Interface/FV-1_Interface.sch (KiCad schematic (older format))
At the start: 29 parts, among them J1 ERK_PWR, J2 TP_GND, J4 IN, J5 OUT, J6 FX_OUT, J7 FX_IN, U2 TL072

Commit message: FV-1 Interface module
Parts:
- removed D2: RED, LED_THT:LED_D3.0mm, symbol Device:LED
- removed D4: BLUE, LED_THT:LED_D3.0mm, symbol Device:LED
- removed J1: ERK_PWR, Connector_IDC:IDC-Header_2x05_P2.54mm_Vertical, symbol Connector_Generic:Conn_02x05_Odd_Even
- removed R1, R3: 3.3k, Resistor_THT:R_Axial_DIN0207_L6.3mm_D2.5mm_P10.16mm_Horizontal, symbol Device:R
- added J1: PWR, Connector_PinHeader_2.54mm:PinHeader_1x03_P2.54mm_Vertical, symbol Connector_Generic:Conn_01x03
- C1, C5: footprint Capacitor_THT:CP_Radial_D6.3mm_P2.50mm -> Capacitor_THT:CP_Radial_D5.0mm_P2.50mm
Connections:
- net +12V: now also J1.1 (Pin_1)
- net -12V: now also J1.3 (Pin_3)
- net GND: now also C1.2, C5.1, J1.2 (Pin_2)
- no-connect marks 7 -> 0
Other:
- moved on the sheet: C1, C10, C5, C6, C7, C8, C9, H1, H2, H3, H4, J2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
